File: Recovery/ejection-test-computer-pcb/ejection-test-pcb/_autosave-ejection-test-pcb.kicad_sch (KiCad schematic)
At the start: 22 parts, among them J1 BATTERY_TERMINAL, J2 LOAD_CELL_CONNECTOR, J3 NICHROME-TERMINAL, Q1 IRLZ34N, SW1 ON, U1 HX7111, U2 LM2596, U3 ESP32_DEVKIT

Commit message: added paho-mqtt-client for test app
Parts:
- gave numbers to parts that had none: 1
Changed lines of the file:
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@@
   (symbol (lib_id "Connector:Micro_SD_Card_Det") (at 142.24 173.99 0) (unit 1)
     (in_bom yes) (on_board yes) (fields_autoplaced)
-    (property "Reference" "J?" (id 0) (at 142.875 152.4 0))
+    (property "Reference" "J4" (id 0) (at 142.875 152.4 0))
     (property "Value" "Micro_SD_Card_Det" (id 1) (at 142.875 154.94 0))
     (property "Footprint" "" (id 2) (at 194.31 156.21 0)
@@
     )
     (path "/ab348d08-997e-4cc6-a582-90b9e2626bcc"
-      (reference "J?") (unit 1) (value "Micro_SD_Card_Det") (footprint "")
+      (reference "J4") (unit 1) (value "Micro_SD_Card_Det") (footprint "")
     )
     (path "/5b7189bd-e7fc-4d66-b9af-d65b01750a9c"
